Commit message: Update workcell.xacro

File: src/myworkcell_core/urdf/workcell.xacro (robot description, xacro)
@@ -4,4 +4,8 @@
 <!-- git clone https://github.com/ros-industrial/universal_robot.git  -->
 <!-- http://ros-industrial.github.io/industrial_training/_source/session3/Workcell-XACRO.html -->
+  <!-- grinder traj -->
+  <xacro:include filename="$(find myworkcell_core)/urdf/grinder.xacro" />
+  <!-- puzzle tool -->
+  <xacro:include filename="$(find myworkcell_core)/urdf/puzzle_mount.xacro" />
 <!-- Add the world frame as a "virtual link" (no geometry) -->
   <link name="world"/>
@@ -29,4 +33,10 @@
     <origin xyz="0 0 0.5" rpy="0 0 0"/>
   </joint>
+<!-- world  to grinder-->
+  <joint name="world_to_grinder" type="fixed">
+    <parent link="world"/>
+    <child link="grinder_frame"/>
+    <origin xyz="0.0 -0.4 0.6" rpy="0 3.14159 0"/>
+  </joint>
 <!-- world to camera -->
   <joint name="world_to_camera" type="fixed">
@@ -43,3 +53,9 @@
     <origin xyz="0 0 0" rpy="0 0 0"/>
   </joint>
+<!-- robot tool0 to puzzle tool  -->
+  <joint name="robot_tool" type="fixed">
+    <parent link="tool0"/>
+    <child link="ee_mount"/>
+    <origin xyz="0 0 0" rpy="1.5708 0 0"/>
+  </joint>
 </robot>
